Commit message: [feat] set mod by Game controller

File: legged_examples/legged_unitree/legged_unitree_description/urdf/robot.xacro (robot description, xacro)
@@ -7,6 +7,6 @@
     <xacro:include filename="$(find legged_unitree_description)/urdf/common/imu.xacro"/>
     <xacro:include filename="$(find legged_unitree_description)/urdf/$(arg robot_type)/const.xacro"/>
-<!--    <xacro:property name="mesh_path" value="../meshes"/>-->
-    <xacro:property name="mesh_path" value="$(find legged_unitree_description)/meshes/$(arg robot_type)"/>
+    <!-- package:// so RViz resolves meshes via rospack (portable across machines/containers) -->
+    <xacro:property name="mesh_path" value="package://legged_unitree_description/meshes/$(arg robot_type)"/>
     <link name="base">
         <visual>
