Commit message: [bug] Controlled divergence a1 and lr_pro

File: legged_robots/lr_pro/lr_pro_description/robot.xacro (robot description, xacro)
@@ -1,1083 +1,49 @@
-<robot name="lr_pro" xmlns:xacro="http://www.ros.org/wiki/xacro">
-  <xacro:arg name="ROBOT" default="lr_pro" />
-  <xacro:include filename="gazebo.xacro" />
-  <!--  <?xml version="1.0" encoding="utf-8"?>-->
-  <link
-          name="base_link">
-    <inertial>
-      <origin
-              xyz="0.0036196 0.0020766 0.014291"
-              rpy="0 0 0" />
-      <mass
-              value="41.55318666" />
-      <inertia
-              ixx="0.36609753"
-              ixy="-0.00244571"
-              ixz="-0.06601466"
-              iyy="1.65137460"
-              iyz="0.00028196"
-              izz="1.78840665" />
-    </inertial>
-    <visual>
-      <origin
-              xyz="0 0 0"
-              rpy="0 0 0" />
-      <geometry>
-        <!-- <mesh filename="../meshes/base_link.STL" /> -->
-         <box size="0.4 0.2 0.15"/>
-      </geometry>
-      <material
-              name="">
-        <color
-                rgba="0.75294 0.75294 0.75294 1" />
-      </material>
-    </visual>
-    <collision>
-      <origin
-              xyz="0 0 0"
-              rpy="0 0 0" />
-      <geometry>
-        <!-- <mesh filename="../meshes/base_link.STL" /> -->
-         <box size="0.4 0.2 0.15"/>
-      </geometry>
-    </collision>
-  </link>
-  <joint name="imu_joint" type="fixed">
-    <parent link="base_link" />
-    <child link="imu_link" />
-    <origin rpy="0 0 0" xyz="33.4e-3 -17.2765e-3 51.0469e-3" />
-  </joint>
-  <link name="imu_link">
-    <inertial>
-      <mass value="0.001" />
-      <origin rpy="0 0 0" xyz="0 0 0" />
-      <inertia ixx="0.0001" ixy="0" ixz="0" iyy="0.0001" iyz="0" izz="0.0001" />
-    </inertial>
-    <visual>
-      <origin rpy="0 0 0" xyz="0 0 0" />
-      <geometry>
-        <box size="0.001 0.001 0.001" />
-      </geometry>
-    </visual>
-    <collision>
-      <origin rpy="0 0 0" xyz="0 0 0" />
-      <geometry>
-        <box size=".001 .001 .001" />
-      </geometry>
-    </collision>
-  </link>
-  <joint name="camera_joint" type="fixed">
-    <parent link="base_link" />
-    <child link="camera_link" />
-    <origin rpy="0 0 0" xyz="0.46 0 0.02" />
-  </joint>
-  <link
-          name="camera_link">
-    <inertial>
-      <mass value="0.001" />
-      <origin rpy="0 0 0" xyz="0 0 0" />
-      <inertia ixx="0.0001" ixy="0" ixz="0" iyy="0.0001" iyz="0" izz="0.0001" />
-    </inertial>
-    <visual>
-      <origin rpy="0 0 0" xyz="0 0 0" />
-      <geometry>
-        <box size="0.001 0.001 0.001" />
-      </geometry>
-    </visual>
-    <collision>
-      <origin rpy="0 0 0" xyz="0 0 0" />
-      <geometry>
-        <box size=".001 .001 .001" />
-      </geometry>
-    </collision>
-  </link>
-  <joint name="livox_joint" type="fixed">
-    <parent link="base_link" />
-    <child link="livox_link" />
-    <origin rpy="0 0 0" xyz="0 0 0.1" />
-  </joint>
-  <link
-          name="livox_link">
-    <inertial>
-      <mass value="0.001" />
-      <origin rpy="0 0 0" xyz="0 0 0" />
-      <inertia ixx="0.0001" ixy="0" ixz="0" iyy="0.0001" iyz="0" izz="0.0001" />
-    </inertial>
-    <visual>
-      <origin rpy="0 0 0" xyz="0 0 0" />
-      <geometry>
-        <box size="0.001 0.001 0.001" />
-      </geometry>
-    </visual>
-    <collision>
-      <origin rpy="0 0 0" xyz="0 0 0" />
-      <geometry>
-        <box size=".001 .001 .001" />
-      </geometry>
-    </collision>
-  </link>
-  <joint name="livox_joint_2" type="fixed">
-    <parent link="base_link" />
-    <child link="livox_link_2" />
-    <origin rpy="0 0.2618 0" xyz="0.5 0 0.1" />
-  </joint>
-  <link
-          name="livox_link_2">
-    <inertial>
-      <mass value="0.001" />
-      <origin rpy="0 0 0" xyz="0 0 0" />
-      <inertia ixx="0.0001" ixy="0" ixz="0" iyy="0.0001" iyz="0" izz="0.0001" />
-    </inertial>
-    <visual>
-      <origin rpy="0 0 0" xyz="0 0 0" />
-      <geometry>
-        <box size="0.001 0.001 0.001" />
-      </geometry>
-    </visual>
-    <collision>
-      <origin rpy="0 0 0" xyz="0 0 0" />
-      <geometry>
-        <box size=".001 .001 .001" />
-      </geometry>
-    </collision>
-  </link>
-  <joint name="lidar_joint" type="fixed">
-    <parent link="base_link" />
-    <child link="lidar_link" />
-    <origin rpy="3.14 0.349 0" xyz="0.5 0 -0.033" />
-  </joint>
-  <link
-          name="lidar_link">
-    <inertial>
-      <mass value="0.001" />
-      <origin rpy="0 0 0" xyz="0 0 0" />
-      <inertia ixx="0.0001" ixy="0" ixz="0" iyy="0.0001" iyz="0" izz="0.0001" />
-    </inertial>
-    <visual>
-      <origin rpy="0 0 0" xyz="0 0 0" />
-      <geometry>
-        <box size="0.001 0.001 0.001" />
-      </geometry>
-    </visual>
-    <collision>
-      <origin rpy="0 0 0" xyz="0 0 0" />
-      <geometry>
-        <box size=".001 .001 .001" />
-      </geometry>
-    </collision>
-  </link>
-  <joint name="lidar2_joint" type="fixed">
-    <parent link="base_link" />
-    <child link="lidar2_link" />
-    <origin rpy="3.14 0.1745 3.14 " xyz="-0.535 0 -0.033" />
-  </joint>
-  <link
-          name="lidar2_link">
-    <inertial>
-      <mass value="0.001" />
-      <origin rpy="0 0 0" xyz="0 0 0" />
-      <inertia ixx="0.0001" ixy="0" ixz="0" iyy="0.0001" iyz="0" izz="0.0001" />
-    </inertial>
-    <visual>
-      <origin rpy="0 0 0" xyz="0 0 0" />
-      <geometry>
-        <box size="0.001 0.001 0.001" />
-      </geometry>
-    </visual>
-    <collision>
-      <origin rpy="0 0 0" xyz="0 0 0" />
-      <geometry>
-        <box size=".001 .001 .001" />
-      </geometry>
-    </collision>
-  </link>
-  <joint name="lidar3_joint" type="fixed">
-    <parent link="base_link" />
-    <child link="lidar3_link" />
-    <origin rpy="0 1.57 0" xyz="-0.25 0 -0.1" />
-  </joint>
-  <link
-          name="lidar3_link">
-    <inertial>
-      <mass value="0.001" />
-      <origin rpy="0 0 0" xyz="0 0 0" />
-      <inertia ixx="0.0001" ixy="0" ixz="0" iyy="0.0001" iyz="0" izz="0.0001" />
-    </inertial>
-    <visual>
-      <origin rpy="0 0 0" xyz="0 0 0" />
-      <geometry>
-        <box size="0.001 0.001 0.001" />
-      </geometry>
-    </visual>
-    <collision>
-      <origin rpy="0 0 0" xyz="0 0 0" />
-      <geometry>
-        <box size=".001 .001 .001" />
-      </geometry>
-    </collision>
-  </link>
-  <link
-          name="FL_hip">
-    <inertial>
-      <origin
-              xyz="0.059894 0.012203 -2.491E-05"
-              rpy="0 0 0" />
-      <mass
-              value="3.14861814" />
-      <inertia
-              ixx="0.00150762"
-              ixy="0.00003652"
-              ixz="0.00000078"
-              iyy="0.00308821"
-              iyz="-0.00000116"
-              izz="0.00282044" />
-    </inertial>
-    <visual>
-      <origin
-              xyz="0 0 0"
-              rpy="0 0 0" />
-      <geometry>
-        <mesh
-                filename="file://$(find lr_pro_description)/meshs_simpilfy/FL_hip.STL" />
-      </geometry>
-      <material
-              name="">
-        <color
-                rgba="0.75294 0.75294 0.75294 1" />
-      </material>
-    </visual>
-    <collision>
-      <origin
-              xyz="0 0 0"
-              rpy="0 0 0" />
-      <geometry>
-        <mesh
-                filename="file://$(find lr_pro_description)/meshs_simpilfy/FL_hip.STL" />
-      </geometry>
-    </collision>
-  </link>
-  <joint
-          name="FL_hip_joint"
-          type="revolute">
-    <origin
-            xyz="0.259 0.072 0"
-            rpy="0 0 0" />
-    <parent
-            link="base_link" />
-    <child
-            link="FL_hip" />
-    <axis
-            xyz="1 0 0" />
-    <limit lower="-0.698" upper="0.698" effort="350" velocity="15" />
-  </joint>
-  <link
-          name="FL_thigh">
-    <inertial>
-      <origin
-              xyz="-0.0095977 0.11103 -0.088387"
-              rpy="0 0 0" />
-      <mass
-              value="4.62267861" />
-      <inertia
-              ixx="0.05234465"
-              ixy="0.00083785"
-              ixz="-0.00317648"
-              iyy="0.04965056"
-              iyz="0.00756963"
-              izz="0.00794928" />
-    </inertial>
-    <visual>
-      <origin
-              xyz="0 0 0"
-              rpy="0 0 0" />
-      <geometry>
-        <mesh
-                filename="file://$(find lr_pro_description)/meshs_simpilfy/FL_thigh.STL" />
-      </geometry>
-      <material
-              name="">
-        <color
-                rgba="0.75294 0.75294 0.75294 1" />
-      </material>
-    </visual>
-    <collision>
-      <origin
-              xyz="0 0 0"
-              rpy="0 0 0" />
-      <geometry>
-        <mesh
-                filename="file://$(find lr_pro_description)/meshs_simpilfy/FL_thigh.STL" />
-      </geometry>
-    </collision>
-  </link>
-  <joint
-          name="FL_thigh_joint"
-          type="revolute">
-    <origin
-            xyz="0.089 0.0395 0"
-            rpy="0 0 0" />
-    <parent
-            link="FL_hip" />
-    <child
-            link="FL_thigh" />
-    <axis
-            xyz="0 1 0" />
-    <limit lower="-2.840" upper="2.840" effort="350" velocity="15" />
-  </joint>
-  <link
-          name="FL_calf">
-    <inertial>
-      <origin
-              xyz="0.02051 8.2897E-06 -0.17043"
-              rpy="0 0 0" />
-      <mass
-              value="0.65025" />
-      <inertia
-              ixx="0.01003897"
-              ixy="0.00000002"
-              ixz="0.00071564"
-              iyy="0.01022625"
-              iyz="-0.00000074"
-              izz="0.00032368" />
-    </inertial>
-    <visual>
-      <origin
-              xyz="0 0 0"
-              rpy="0 0 0" />
-      <geometry>
-        <mesh
-                filename="file://$(find lr_pro_description)/meshs_simpilfy/FL_calf.STL" />
-      </geometry>
-      <material
-              name="">
-        <color
-                rgba="0.75294 0.75294 0.75294 1" />
-      </material>
-    </visual>
-    <collision>
-      <origin
-              xyz="0 0 0"
-              rpy="0 0 0" />
-      <geometry>
-        <mesh
-                filename="file://$(find lr_pro_description)/meshs_simpilfy/FL_calf.STL" />
-      </geometry>
-    </collision>
-  </link>
-  <joint
-          name="FL_calf_joint"
-          type="revolute">
-    <origin
-            xyz="0 0.1323 -0.35"
-            rpy="0 0 0" />
-    <parent
-            link="FL_thigh" />
-    <child
-            link="FL_calf" />
-    <axis
-            xyz="0 1 0" />
-    <limit lower="-2.76634" upper="-0.68067" effort="350" velocity="15" />
-  </joint>
-  <link
-          name="FL_foot">
-    <inertial>
-      <origin
-              xyz="-0.0068215 5.1068E-08 -0.0064099"
-              rpy="0 0 0" />
-      <mass
-              value="0.17599" />
-      <inertia
-              ixx="0.00011789"
-              ixy="0.00000000"
-              ixz="0.00002693"
-              iyy="0.00011149"
-              iyz="0.00000000"
-              izz="0.00011428" />
-    </inertial>
-    <visual>
-      <origin
-              xyz="0 0 0"
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
File: legged_robots/lr_pro/lr_pro_description/urdf/lr_pro/const.xacro (robot description, xacro)
@@ -1,12 +1,12 @@
 <?xml version="1.0"?>
 <robot xmlns:xacro="http://www.ros.org/wiki/xacro" name="lr_pro_description">
-    <!-- Constants for robot dimensions -->
+    <!-- 机器人尺寸常量 -->
     <xacro:property name="stick_mass" value="0.00001"/>
-    <!-- simplified collision value: from base_link box size="0.4 0.2 0.15" -->
+    <!-- 简化碰撞体尺寸：来自 base_link 的 box size="0.4 0.2 0.15" -->
     <xacro:property name="trunk_length" value="0.4"/>
     <xacro:property name="trunk_width" value="0.2"/>
     <xacro:property name="trunk_height" value="0.15"/>
-    <!-- These are kept for compatibility with A1-style macros.
-         lr_pro uses mesh collision for hip/thigh/calf, so these are fallback values. -->
+    <!-- 保留这些参数是为了兼容 A1 风格的通用宏。
+         lr_pro 的 hip/thigh/calf 使用 mesh 碰撞体时，这些值作为备用参数。 -->
     <xacro:property name="hip_radius" value="0.046"/>
     <xacro:property name="hip_length" value="0.04"/>
@@ -20,40 +20,40 @@
     <xacro:property name="calf_height" value="0.016"/>
     <xacro:property name="calf_x_offset" value="0.0"/>
-    <!-- from foot collision sphere radius="0.042" -->
+    <!-- 来自足端碰撞球半径 radius="0.042" -->
     <xacro:property name="foot_radius" value="0.042"/>
-    <!-- kinematic value -->
-    <!-- from FL/RL calf joint origin xyz="0 0.1323 -0.35" -->
+    <!-- 运动学参数 -->
+    <!-- 来自 FL/RL 小腿关节 origin xyz="0 0.1323 -0.35" -->
     <xacro:property name="thigh_offset" value="0.1323"/>
     <xacro:property name="thigh_length" value="0.35"/>
-    <!-- from foot_fixed origin xyz="0 0 -0.35" -->
+    <!-- 来自 foot_fixed 关节 origin xyz="0 0 -0.35" -->
     <xacro:property name="calf_length" value="0.35"/>
-    <!-- leg offset from trunk center value -->
-    <!-- from FL/FR/RL/RR hip joint origin xyz="+-0.259 +-0.072 0" -->
+    <!-- 腿部相对机身中心的偏移量 -->
+    <!-- 来自 FL/FR/RL/RR 髋关节 origin xyz="+-0.259 +-0.072 0" -->
     <xacro:property name="leg_offset_x" value="0.259"/>
     <xacro:property name="leg_offset_y" value="0.072"/>
     <xacro:property name="trunk_offset_z" value="0.0"/>
-    <!-- from thigh joint origin xyz="+-0.089 +-0.0395 0" -->
+    <!-- 来自大腿关节 origin xyz="+-0.089 +-0.0395 0" -->
     <xacro:property name="hip_offset_x" value="0.089"/>
     <xacro:property name="hip_offset" value="0.0395"/>
-    <!-- joint limits -->
+    <!-- 关节限位 -->
     <xacro:property name="damping" value="0"/>
     <xacro:property name="friction" value="0"/>
-    <!-- HAA / hip joint: lower="-0.698" upper="0.698" effort="350" velocity="15" -->
+    <!-- HAA / 髋外展关节：lower="-0.698" upper="0.698" effort="350" velocity="15" -->
     <xacro:property name="hip_position_max" value="0.698"/>
     <xacro:property name="hip_position_min" value="-0.698"/>
     <xacro:property name="hip_velocity_max" value="15"/>
     <xacro:property name="hip_torque_max" value="350"/>
-    <!-- HFE / thigh joint: lower="-2.840" upper="2.840" effort="350" velocity="15" -->
+    <!-- HFE / 髋俯仰关节：lower="-2.840" upper="2.840" effort="350" velocity="15" -->
     <xacro:property name="thigh_position_max" value="2.840"/>
     <xacro:property name="thigh_position_min" value="-2.840"/>
     <xacro:property name="thigh_velocity_max" value="15"/>
     <xacro:property name="thigh_torque_max" value="350"/>
-    <!-- KFE / calf joint: lower="-2.76634" upper="-0.68067" effort="350" velocity="15" -->
+    <!-- KFE / 膝关节：lower="-2.76634" upper="-0.68067" effort="350" velocity="15" -->
     <xacro:property name="calf_position_max" value="-0.68067"/>
     <xacro:property name="calf_position_min" value="-2.76634"/>
     <xacro:property name="calf_velocity_max" value="15"/>
     <xacro:property name="calf_torque_max" value="350"/>
-    <!-- dynamics inertial value -->
-    <!-- trunk / base_link -->
+    <!-- 动力学惯性参数 -->
+    <!-- 机身 / base_link -->
     <xacro:property name="trunk_mass" value="41.55318666"/>
     <xacro:property name="trunk_com_x" value="0.0036196"/>
@@ -66,5 +66,5 @@
     <xacro:property name="trunk_iyz" value="0.00028196"/>
     <xacro:property name="trunk_izz" value="1.78840665"/>
-    <!-- hip: using FL_hip as template -->
+    <!-- 髋部：以 FL_hip 作为模板 -->
     <xacro:property name="hip_mass" value="3.14861814"/>
     <xacro:property name="hip_com_x" value="0.059894"/>
@@ -77,5 +77,5 @@
     <xacro:property name="hip_iyz" value="-0.00000116"/>
     <xacro:property name="hip_izz" value="0.00282044"/>
-    <!-- thigh: using FL_thigh as template -->
+    <!-- 大腿：以 FL_thigh 作为模板 -->
     <xacro:property name="thigh_mass" value="4.62267861"/>
     <xacro:property name="thigh_com_x" value="-0.0095977"/>
@@ -88,5 +88,5 @@
     <xacro:property name="thigh_iyz" value="0.00756963"/>
     <xacro:property name="thigh_izz" value="0.00794928"/>
-    <!-- calf -->
+    <!-- 小腿 -->
     <xacro:property name="calf_mass" value="0.65024748"/>
     <xacro:property name="calf_com_x" value="0.02051"/>
@@ -99,5 +99,5 @@
     <xacro:property name="calf_iyz" value="-0.00000074"/>
     <xacro:property name="calf_izz" value="0.00032368"/>
-    <!-- foot -->
+    <!-- 足端 -->
     <xacro:property name="foot_mass" value="0.17599179"/>
     <xacro:property name="foot_com_x" value="-0.0068215"/>
@@ -110,5 +110,5 @@
     <xacro:property name="foot_iyz" value="0.0"/>
     <xacro:property name="foot_izz" value="0.00011428"/>
-    <!-- sensor extrinsic parameters -->
+    <!-- 传感器外参 -->
     <xacro:property name="imu_x" value="0.0334"/>
     <xacro:property name="imu_y" value="-0.0172765"/>
