Commit message: [add] Add lr_pro mode & could be display

File: legged_robots/lr_pro/lr_pro_description/robot.xacro (robot description, xacro)
@@ -1,5 +1,4 @@
 <robot name="lr_pro" xmlns:xacro="http://www.ros.org/wiki/xacro">
   <xacro:arg name="ROBOT" default="lr_pro" />
-  <xacro:include filename="gazebo.xacro" />
   <!--  <?xml version="1.0" encoding="utf-8"?>-->
   <link
@@ -24,6 +23,5 @@
               rpy="0 0 0" />
       <geometry>
-        <!-- <mesh filename="../meshes/base_link.STL" /> -->
-         <box size="0.4 0.2 0.15"/>
+        <mesh filename="file://$(find lr_pro_description)/meshes/base_link.STL" />
       </geometry>
       <material
@@ -239,19 +237,19 @@
       <geometry>
         <mesh
-                filename="file://$(find lr_pro_description)/meshs_simpilfy/FL_hip.STL" />
-      </geometry>
-      <material
-              name="">
-        <color
-                rgba="0.75294 0.75294 0.75294 1" />
-      </material>
-    </visual>
-    <collision>
-      <origin
-              xyz="0 0 0"
-              rpy="0 0 0" />
-      <geometry>
-        <mesh
-                filename="file://$(find lr_pro_description)/meshs_simpilfy/FL_hip.STL" />
+                filename="file://$(find lr_pro_description)/meshes/FL_hip.STL" />
+      </geometry>
+      <material
+              name="">
+        <color
+                rgba="0.75294 0.75294 0.75294 1" />
+      </material>
+    </visual>
+    <collision>
+      <origin
+              xyz="0 0 0"
+              rpy="0 0 0" />
+      <geometry>
+        <mesh
+                filename="file://$(find lr_pro_description)/meshes/FL_hip.STL" />
       </geometry>
     </collision>
@@ -293,19 +291,19 @@
       <geometry>
         <mesh
-                filename="file://$(find lr_pro_description)/meshs_simpilfy/FL_thigh.STL" />
-      </geometry>
-      <material
-              name="">
-        <color
-                rgba="0.75294 0.75294 0.75294 1" />
-      </material>
-    </visual>
-    <collision>
-      <origin
-              xyz="0 0 0"
-              rpy="0 0 0" />
-      <geometry>
-        <mesh
-                filename="file://$(find lr_pro_description)/meshs_simpilfy/FL_thigh.STL" />
+                filename="file://$(find lr_pro_description)/meshes/FL_thigh.STL" />
+      </geometry>
+      <material
+              name="">
+        <color
+                rgba="0.75294 0.75294 0.75294 1" />
+      </material>
+    </visual>
+    <collision>
+      <origin
+              xyz="0 0 0"
+              rpy="0 0 0" />
+      <geometry>
+        <mesh
+                filename="file://$(find lr_pro_description)/meshes/FL_thigh.STL" />
       </geometry>
     </collision>
@@ -347,19 +345,19 @@
       <geometry>
         <mesh
-                filename="file://$(find lr_pro_description)/meshs_simpilfy/FL_calf.STL" />
-      </geometry>
-      <material
-              name="">
-        <color
-                rgba="0.75294 0.75294 0.75294 1" />
-      </material>
-    </visual>
-    <collision>
-      <origin
-              xyz="0 0 0"
-              rpy="0 0 0" />
-      <geometry>
-        <mesh
-                filename="file://$(find lr_pro_description)/meshs_simpilfy/FL_calf.STL" />
+                filename="file://$(find lr_pro_description)/meshes/FL_calf.STL" />
+      </geometry>
+      <material
+              name="">
+        <color
+                rgba="0.75294 0.75294 0.75294 1" />
+      </material>
+    </visual>
+    <collision>
+      <origin
+              xyz="0 0 0"
+              rpy="0 0 0" />
+      <geometry>
+        <mesh
+                filename="file://$(find lr_pro_description)/meshes/FL_calf.STL" />
       </geometry>
     </collision>
@@ -401,5 +399,5 @@
       <geometry>
         <mesh
-                filename="file://$(find lr_pro_description)/meshs_simpilfy/FL_foot.STL" />
+                filename="file://$(find lr_pro_description)/meshes/FL_foot.STL" />
       </geometry>
       <material
@@ -454,19 +452,19 @@
       <geometry>
         <mesh
-                filename="file://$(find lr_pro_description)/meshs_simpilfy/FR_hip.STL" />
-      </geometry>
-      <material
-              name="">
-        <color
-                rgba="0.75294 0.75294 0.75294 1" />
-      </material>
-    </visual>
-    <collision>
-      <origin
-              xyz="0 0 0"
-              rpy="0 0 0" />
-      <geometry>
-        <mesh
-                filename="file://$(find lr_pro_description)/meshs_simpilfy/FR_hip.STL" />
+                filename="file://$(find lr_pro_description)/meshes/FR_hip.STL" />
+      </geometry>
+      <material
+              name="">
+        <color
+                rgba="0.75294 0.75294 0.75294 1" />
+      </material>
+    </visual>
+    <collision>
+      <origin
+              xyz="0 0 0"
+              rpy="0 0 0" />
+      <geometry>
+        <mesh
+                filename="file://$(find lr_pro_description)/meshes/FR_hip.STL" />
       </geometry>
     </collision>
@@ -508,19 +506,19 @@
       <geometry>
         <mesh
-                filename="file://$(find lr_pro_description)/meshs_simpilfy/FR_thigh.STL" />
-      </geometry>
-      <material
-              name="">
-        <color
-                rgba="0.75294 0.75294 0.75294 1" />
-      </material>
-    </visual>
-    <collision>
-      <origin
-              xyz="0 0 0"
-              rpy="0 0 0" />
-      <geometry>
-        <mesh
-                filename="file://$(find lr_pro_description)/meshs_simpilfy/FR_thigh.STL" />
+                filename="file://$(find lr_pro_description)/meshes/FR_thigh.STL" />
+      </geometry>
+      <material
+              name="">
+        <color
+                rgba="0.75294 0.75294 0.75294 1" />
+      </material>
+    </visual>
+    <collision>
+      <origin
+              xyz="0 0 0"
+              rpy="0 0 0" />
+      <geometry>
+        <mesh
+                filename="file://$(find lr_pro_description)/meshes/FR_thigh.STL" />
       </geometry>
     </collision>
@@ -562,19 +560,19 @@
       <geometry>
         <mesh
-                filename="file://$(find lr_pro_description)/meshs_simpilfy/FR_calf.STL" />
-      </geometry>
-      <material
-              name="">
-        <color
-                rgba="0.75294 0.75294 0.75294 1" />
-      </material>
-    </visual>
-    <collision>
-      <origin
-              xyz="0 0 0"
-              rpy="0 0 0" />
-      <geometry>
-        <mesh
-                filename="file://$(find lr_pro_description)/meshs_simpilfy/FR_calf.STL" />
+                filename="file://$(find lr_pro_description)/meshes/FR_calf.STL" />
+      </geometry>
+      <material
+              name="">
+        <color
+                rgba="0.75294 0.75294 0.75294 1" />
+      </material>
+    </visual>
+    <collision>
+      <origin
+              xyz="0 0 0"
+              rpy="0 0 0" />
+      <geometry>
+        <mesh
+                filename="file://$(find lr_pro_description)/meshes/FR_calf.STL" />
       </geometry>
     </collision>
@@ -616,5 +614,5 @@
       <geometry>
         <mesh
-                filename="file://$(find lr_pro_description)/meshs_simpilfy/FR_foot.STL" />
+                filename="file://$(find lr_pro_description)/meshes/FR_foot.STL" />
       </geometry>
       <material
@@ -669,19 +667,19 @@
       <geometry>
         <mesh
-                filename="file://$(find lr_pro_description)/meshs_simpilfy/RL_hip.STL" />
-      </geometry>
-      <material
-              name="">
-        <color
-                rgba="0.75294 0.75294 0.75294 1" />
-      </material>
-    </visual>
-    <collision>
-      <origin
-              xyz="0 0 0"
-              rpy="0 0 0" />
-      <geometry>
-        <mesh
-                filename="file://$(find lr_pro_description)/meshs_simpilfy/RL_hip.STL" />
+                filename="file://$(find lr_pro_description)/meshes/RL_hip.STL" />
+      </geometry>
+      <material
+              name="">
+        <color
+                rgba="0.75294 0.75294 0.75294 1" />
+      </material>
+    </visual>
+    <collision>
+      <origin
+              xyz="0 0 0"
+              rpy="0 0 0" />
+      <geometry>
+        <mesh
+                filename="file://$(find lr_pro_description)/meshes/RL_hip.STL" />
       </geometry>
     </collision>
@@ -723,19 +721,19 @@
       <geometry>
         <mesh
-                filename="file://$(find lr_pro_description)/meshs_simpilfy/RL_thigh.STL" />
-      </geometry>
-      <material
-              name="">
-        <color
-                rgba="0.75294 0.75294 0.75294 1" />
-      </material>
-    </visual>
-    <collision>
-      <origin
-              xyz="0 0 0"
-              rpy="0 0 0" />
-      <geometry>
-        <mesh
-                filename="file://$(find lr_pro_description)/meshs_simpilfy/RL_thigh.STL" />
+                filename="file://$(find lr_pro_description)/meshes/RL_thigh.STL" />
+      </geometry>
+      <material
+              name="">
+        <color
+                rgba="0.75294 0.75294 0.75294 1" />
+      </material>
+    </visual>
+    <collision>
+      <origin
+              xyz="0 0 0"
+              rpy="0 0 0" />
+      <geometry>
+        <mesh
+                filename="file://$(find lr_pro_description)/meshes/RL_thigh.STL" />
       </geometry>
     </collision>
@@ -777,19 +775,19 @@
       <geometry>
         <mesh
-                filename="file://$(find lr_pro_description)/meshs_simpilfy/RL_calf.STL" />
-      </geometry>
-      <material
-              name="">
-        <color
-                rgba="0.75294 0.75294 0.75294 1" />
-      </material>
-    </visual>
-    <collision>
-      <origin
-              xyz="0 0 0"
-              rpy="0 0 0" />
-      <geometry>
-        <mesh
-                filename="file://$(find lr_pro_description)/meshs_simpilfy/RL_calf.STL" />
+                filename="file://$(find lr_pro_description)/meshes/RL_calf.STL" />
+      </geometry>
+      <material
+              name="">
+        <color
+                rgba="0.75294 0.75294 0.75294 1" />
+      </material>
+    </visual>
+    <collision>
+      <origin
+              xyz="0 0 0"
+              rpy="0 0 0" />
+      <geometry>
+        <mesh
+                filename="file://$(find lr_pro_description)/meshes/RL_calf.STL" />
       </geometry>
     </collision>
@@ -831,5 +829,5 @@
       <geometry>
         <mesh
-                filename="file://$(find lr_pro_description)/meshs_simpilfy/RL_foot.STL" />
+                filename="file://$(find lr_pro_description)/meshes/RL_foot.STL" />
       </geometry>
       <material
@@ -884,19 +882,19 @@
       <geometry>
         <mesh
-                filename="file://$(find lr_pro_description)/meshs_simpilfy/RR_hip.STL" />
-      </geometry>
-      <material
-              name="">
-        <color
-                rgba="0.75294 0.75294 0.75294 1" />
-      </material>
-    </visual>
-    <collision>
-      <origin
-              xyz="0 0 0"
-              rpy="0 0 0" />
-      <geometry>
-        <mesh
-                filename="file://$(find lr_pro_description)/meshs_simpilfy/RR_hip.STL" />
+                filename="file://$(find lr_pro_description)/meshes/RR_hip.STL" />
+      </geometry>
+      <material
+              name="">
+        <color
+                rgba="0.75294 0.75294 0.75294 1" />
+      </material>
+    </visual>
+    <collision>
+      <origin
+              xyz="0 0 0"
+              rpy="0 0 0" />
+      <geometry>
+        <mesh
+                filename="file://$(find lr_pro_description)/meshes/RR_hip.STL" />
       </geometry>
     </collision>
@@ -938,19 +936,19 @@
       <geometry>
         <mesh
-                filename="file://$(find lr_pro_description)/meshs_simpilfy/RR_thigh.STL" />
-      </geometry>
-      <material
-              name="">
-        <color
-                rgba="0.75294 0.75294 0.75294 1" />
-      </material>
-    </visual>
-    <collision>
-      <origin
-              xyz="0 0 0"
-              rpy="0 0 0" />
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