Commit message: [bug] lr_pro had a problem with his standing posture, which caused him to fall. It is tentatively determined to be a problem with the order in which he jointed his feet.

File: legged_robots/lr_pro/lr_pro_description/robot.xacro (robot description, xacro)
@@ -1,1081 +1,50 @@
-<robot name="lr_pro" xmlns:xacro="http://www.ros.org/wiki/xacro">
-  <xacro:arg name="ROBOT" default="lr_pro" />
-  <!--  <?xml version="1.0" encoding="utf-8"?>-->
-  <link
-          name="base_link">
-    <inertial>
-      <origin
-              xyz="0.0036196 0.0020766 0.014291"
-              rpy="0 0 0" />
-      <mass
-              value="41.55318666" />
-      <inertia
-              ixx="0.36609753"
-              ixy="-0.00244571"
-              ixz="-0.06601466"
-              iyy="1.65137460"
-              iyz="0.00028196"
-              izz="1.78840665" />
-    </inertial>
-    <visual>
-      <origin
-              xyz="0 0 0"
-              rpy="0 0 0" />
-      <geometry>
-        <mesh filename="file://$(find lr_pro_description)/meshes/base_link.STL" />
-      </geometry>
-      <material
-              name="">
-        <color
-                rgba="0.75294 0.75294 0.75294 1" />
-      </material>
-    </visual>
-    <collision>
-      <origin
-              xyz="0 0 0"
-              rpy="0 0 0" />
-      <geometry>
-        <!-- <mesh filename="../meshes/base_link.STL" /> -->
-         <box size="0.4 0.2 0.15"/>
-      </geometry>
-    </collision>
-  </link>
-  <joint name="imu_joint" type="fixed">
-    <parent link="base_link" />
-    <child link="imu_link" />
-    <origin rpy="0 0 0" xyz="33.4e-3 -17.2765e-3 51.0469e-3" />
-  </joint>
-  <link name="imu_link">
-    <inertial>
-      <mass value="0.001" />
-      <origin rpy="0 0 0" xyz="0 0 0" />
-      <inertia ixx="0.0001" ixy="0" ixz="0" iyy="0.0001" iyz="0" izz="0.0001" />
-    </inertial>
-    <visual>
-      <origin rpy="0 0 0" xyz="0 0 0" />
-      <geometry>
-        <box size="0.001 0.001 0.001" />
-      </geometry>
-    </visual>
-    <collision>
-      <origin rpy="0 0 0" xyz="0 0 0" />
-      <geometry>
-        <box size=".001 .001 .001" />
-      </geometry>
-    </collision>
-  </link>
-  <joint name="camera_joint" type="fixed">
-    <parent link="base_link" />
-    <child link="camera_link" />
-    <origin rpy="0 0 0" xyz="0.46 0 0.02" />
-  </joint>
-  <link
-          name="camera_link">
-    <inertial>
-      <mass value="0.001" />
-      <origin rpy="0 0 0" xyz="0 0 0" />
-      <inertia ixx="0.0001" ixy="0" ixz="0" iyy="0.0001" iyz="0" izz="0.0001" />
-    </inertial>
-    <visual>
-      <origin rpy="0 0 0" xyz="0 0 0" />
-      <geometry>
-        <box size="0.001 0.001 0.001" />
-      </geometry>
-    </visual>
-    <collision>
-      <origin rpy="0 0 0" xyz="0 0 0" />
-      <geometry>
-        <box size=".001 .001 .001" />
-      </geometry>
-    </collision>
-  </link>
-  <joint name="livox_joint" type="fixed">
-    <parent link="base_link" />
-    <child link="livox_link" />
-    <origin rpy="0 0 0" xyz="0 0 0.1" />
-  </joint>
-  <link
-          name="livox_link">
-    <inertial>
-      <mass value="0.001" />
-      <origin rpy="0 0 0" xyz="0 0 0" />
-      <inertia ixx="0.0001" ixy="0" ixz="0" iyy="0.0001" iyz="0" izz="0.0001" />
-    </inertial>
-    <visual>
-      <origin rpy="0 0 0" xyz="0 0 0" />
-      <geometry>
-        <box size="0.001 0.001 0.001" />
-      </geometry>
-    </visual>
-    <collision>
-      <origin rpy="0 0 0" xyz="0 0 0" />
-      <geometry>
-        <box size=".001 .001 .001" />
-      </geometry>
-    </collision>
-  </link>
-  <joint name="livox_joint_2" type="fixed">
-    <parent link="base_link" />
-    <child link="livox_link_2" />
-    <origin rpy="0 0.2618 0" xyz="0.5 0 0.1" />
-  </joint>
-  <link
-          name="livox_link_2">
-    <inertial>
-      <mass value="0.001" />
-      <origin rpy="0 0 0" xyz="0 0 0" />
-      <inertia ixx="0.0001" ixy="0" ixz="0" iyy="0.0001" iyz="0" izz="0.0001" />
-    </inertial>
-    <visual>
-      <origin rpy="0 0 0" xyz="0 0 0" />
-      <geometry>
-        <box size="0.001 0.001 0.001" />
-      </geometry>
-    </visual>
-    <collision>
-      <origin rpy="0 0 0" xyz="0 0 0" />
-      <geometry>
-        <box size=".001 .001 .001" />
-      </geometry>
-    </collision>
-  </link>
-  <joint name="lidar_joint" type="fixed">
-    <parent link="base_link" />
-    <child link="lidar_link" />
-    <origin rpy="3.14 0.349 0" xyz="0.5 0 -0.033" />
-  </joint>
-  <link
-          name="lidar_link">
-    <inertial>
-      <mass value="0.001" />
-      <origin rpy="0 0 0" xyz="0 0 0" />
-      <inertia ixx="0.0001" ixy="0" ixz="0" iyy="0.0001" iyz="0" izz="0.0001" />
-    </inertial>
-    <visual>
-      <origin rpy="0 0 0" xyz="0 0 0" />
-      <geometry>
-        <box size="0.001 0.001 0.001" />
-      </geometry>
-    </visual>
-    <collision>
-      <origin rpy="0 0 0" xyz="0 0 0" />
-      <geometry>
-        <box size=".001 .001 .001" />
-      </geometry>
-    </collision>
-  </link>
-  <joint name="lidar2_joint" type="fixed">
-    <parent link="base_link" />
-    <child link="lidar2_link" />
-    <origin rpy="3.14 0.1745 3.14 " xyz="-0.535 0 -0.033" />
-  </joint>
-  <link
-          name="lidar2_link">
-    <inertial>
-      <mass value="0.001" />
-      <origin rpy="0 0 0" xyz="0 0 0" />
-      <inertia ixx="0.0001" ixy="0" ixz="0" iyy="0.0001" iyz="0" izz="0.0001" />
-    </inertial>
-    <visual>
-      <origin rpy="0 0 0" xyz="0 0 0" />
-      <geometry>
-        <box size="0.001 0.001 0.001" />
-      </geometry>
-    </visual>
-    <collision>
-      <origin rpy="0 0 0" xyz="0 0 0" />
-      <geometry>
-        <box size=".001 .001 .001" />
-      </geometry>
-    </collision>
-  </link>
-  <joint name="lidar3_joint" type="fixed">
-    <parent link="base_link" />
-    <child link="lidar3_link" />
-    <origin rpy="0 1.57 0" xyz="-0.25 0 -0.1" />
-  </joint>
-  <link
-          name="lidar3_link">
-    <inertial>
-      <mass value="0.001" />
-      <origin rpy="0 0 0" xyz="0 0 0" />
-      <inertia ixx="0.0001" ixy="0" ixz="0" iyy="0.0001" iyz="0" izz="0.0001" />
-    </inertial>
-    <visual>
-      <origin rpy="0 0 0" xyz="0 0 0" />
-      <geometry>
-        <box size="0.001 0.001 0.001" />
-      </geometry>
-    </visual>
-    <collision>
-      <origin rpy="0 0 0" xyz="0 0 0" />
-      <geometry>
-        <box size=".001 .001 .001" />
-      </geometry>
-    </collision>
-  </link>
-  <link
-          name="FL_hip">
-    <inertial>
-      <origin
-              xyz="0.059894 0.012203 -2.491E-05"
-              rpy="0 0 0" />
-      <mass
-              value="3.14861814" />
-      <inertia
-              ixx="0.00150762"
-              ixy="0.00003652"
-              ixz="0.00000078"
-              iyy="0.00308821"
-              iyz="-0.00000116"
-              izz="0.00282044" />
-    </inertial>
-    <visual>
-      <origin
-              xyz="0 0 0"
-              rpy="0 0 0" />
-      <geometry>
-        <mesh
-                filename="file://$(find lr_pro_description)/meshes/FL_hip.STL" />
-      </geometry>
-      <material
-              name="">
-        <color
-                rgba="0.75294 0.75294 0.75294 1" />
-      </material>
-    </visual>
-    <collision>
-      <origin
-              xyz="0 0 0"
-              rpy="0 0 0" />
-      <geometry>
-        <mesh
-                filename="file://$(find lr_pro_description)/meshes/FL_hip.STL" />
-      </geometry>
-    </collision>
-  </link>
-  <joint
-          name="FL_hip_joint"
-          type="revolute">
-    <origin
-            xyz="0.259 0.072 0"
-            rpy="0 0 0" />
-    <parent
-            link="base_link" />
-    <child
-            link="FL_hip" />
-    <axis
-            xyz="1 0 0" />
-    <limit lower="-0.698" upper="0.698" effort="350" velocity="15" />
-  </joint>
-  <link
-          name="FL_thigh">
-    <inertial>
-      <origin
-              xyz="-0.0095977 0.11103 -0.088387"
-              rpy="0 0 0" />
-      <mass
-              value="4.62267861" />
-      <inertia
-              ixx="0.05234465"
-              ixy="0.00083785"
-              ixz="-0.00317648"
-              iyy="0.04965056"
-              iyz="0.00756963"
-              izz="0.00794928" />
-    </inertial>
-    <visual>
-      <origin
-              xyz="0 0 0"
-              rpy="0 0 0" />
-      <geometry>
-        <mesh
-                filename="file://$(find lr_pro_description)/meshes/FL_thigh.STL" />
-      </geometry>
-      <material
-              name="">
-        <color
-                rgba="0.75294 0.75294 0.75294 1" />
-      </material>
-    </visual>
-    <collision>
-      <origin
-              xyz="0 0 0"
-              rpy="0 0 0" />
-      <geometry>
-        <mesh
-                filename="file://$(find lr_pro_description)/meshes/FL_thigh.STL" />
-      </geometry>
-    </collision>
-  </link>
-  <joint
-          name="FL_thigh_joint"
-          type="revolute">
-    <origin
-            xyz="0.089 0.0395 0"
-            rpy="0 0 0" />
-    <parent
-            link="FL_hip" />
-    <child
-            link="FL_thigh" />
-    <axis
-            xyz="0 1 0" />
-    <limit lower="-2.840" upper="2.840" effort="350" velocity="15" />
-  </joint>
-  <link
-          name="FL_calf">
-    <inertial>
-      <origin
-              xyz="0.02051 8.2897E-06 -0.17043"
-              rpy="0 0 0" />
-      <mass
-              value="0.65025" />
-      <inertia
-              ixx="0.01003897"
-              ixy="0.00000002"
-              ixz="0.00071564"
-              iyy="0.01022625"
-              iyz="-0.00000074"
-              izz="0.00032368" />
-    </inertial>
-    <visual>
-      <origin
-              xyz="0 0 0"
-              rpy="0 0 0" />
-      <geometry>
-        <mesh
-                filename="file://$(find lr_pro_description)/meshes/FL_calf.STL" />
-      </geometry>
-      <material
-              name="">
-        <color
-                rgba="0.75294 0.75294 0.75294 1" />
-      </material>
-    </visual>
-    <collision>
-      <origin
-              xyz="0 0 0"
-              rpy="0 0 0" />
-      <geometry>
-        <mesh
-                filename="file://$(find lr_pro_description)/meshes/FL_calf.STL" />
-      </geometry>
-    </collision>
-  </link>
-  <joint
-          name="FL_calf_joint"
-          type="revolute">
-    <origin
-            xyz="0 0.1323 -0.35"
-            rpy="0 0 0" />
-    <parent
-            link="FL_thigh" />
-    <child
-            link="FL_calf" />
-    <axis
-            xyz="0 1 0" />
-    <limit lower="-2.76634" upper="-0.68067" effort="350" velocity="15" />
-  </joint>
-  <link
-          name="FL_foot">
-    <inertial>
-      <origin
-              xyz="-0.0068215 5.1068E-08 -0.0064099"
-              rpy="0 0 0" />
-      <mass
-              value="0.17599" />
-      <inertia
-              ixx="0.00011789"
-              ixy="0.00000000"
-              ixz="0.00002693"
-              iyy="0.00011149"
-              iyz="0.00000000"
-              izz="0.00011428" />
-    </inertial>
-    <visual>
-      <origin
-              xyz="0 0 0"
-              rpy="0 0 0" />
-      <geometry>
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
File: legged_robots/lr_pro/lr_pro_description/urdf/common/gazebo.xacro (robot description, xacro)
@@ -3,9 +3,9 @@
     <!-- Gazebo 中加载 ros2_control 插件。
          第一份参数文件声明 controller 类型，第二份可选参数文件覆盖当前机器人专属的 urdfFile、taskFile、referenceFile。 -->
-    <xacro:if value="${enable_gazebo_control == 'true'}">
+    <xacro:if value="${'$(arg enable_gazebo_control)' == 'true'}">
         <gazebo>
         <plugin name="gazebo_ros2_control" filename="libgazebo_ros2_control.so">
             <parameters>$(find legged_controllers)/config/controllers.yaml</parameters>
-            <xacro:if value="${enable_gazebo_control == 'true'}">
+            <xacro:if value="${'$(arg controller_params_file)' != ''}">
                 <parameters>$(arg controller_params_file)</parameters>
             </xacro:if>

File: legged_robots/lr_pro/lr_pro_description/urdf/lr_pro/const.xacro (robot description, xacro)
@@ -39,19 +39,19 @@
     <xacro:property name="damping" value="0"/>
     <xacro:property name="friction" value="0"/>
-    <!-- HAA / hip joint: lower="-0.698" upper="0.698" effort="350" velocity="15" -->
+    <!-- HAA / hip joint: lower="-0.698" upper="0.698" effort="220" velocity="12" -->
     <xacro:property name="hip_position_max" value="0.698"/>
     <xacro:property name="hip_position_min" value="-0.698"/>
-    <xacro:property name="hip_velocity_max" value="15"/>
-    <xacro:property name="hip_torque_max" value="350"/>
-    <!-- HFE / thigh joint: lower="-2.840" upper="2.840" effort="350" velocity="15" -->
+    <xacro:property name="hip_velocity_max" value="12"/>
+    <xacro:property name="hip_torque_max" value="220"/>
+    <!-- HFE / thigh joint: lower="-2.840" upper="2.840" effort="220" velocity="12" -->
     <xacro:property name="thigh_position_max" value="2.840"/>
     <xacro:property name="thigh_position_min" value="-2.840"/>
-    <xacro:property name="thigh_velocity_max" value="15"/>
-    <xacro:property name="thigh_torque_max" value="350"/>
-    <!-- KFE / calf joint: lower="-2.76634" upper="-0.68067" effort="350" velocity="15" -->
+    <xacro:property name="thigh_velocity_max" value="12"/>
+    <xacro:property name="thigh_torque_max" value="220"/>
+    <!-- KFE / calf joint: lower="-2.76634" upper="-0.68067" effort="280" velocity="12" -->
     <xacro:property name="calf_position_max" value="-0.68067"/>
     <xacro:property name="calf_position_min" value="-2.76634"/>
-    <xacro:property name="calf_velocity_max" value="15"/>
-    <xacro:property name="calf_torque_max" value="350"/>
+    <xacro:property name="calf_velocity_max" value="12"/>
+    <xacro:property name="calf_torque_max" value="280"/>
     <!-- dynamics inertial value -->
     <!-- trunk / base_link -->
