Commit message: [change] modify plugin name

File: legged_robots/legged_description/urdf/common/ros2_control.xacro (robot description, xacro)
@@ -18,6 +18,6 @@
         </sensor>
     </xacro:macro>
-    <xacro:macro name="legged_unitree_ros2_control" params="hardware_plugin robot_type power_limit contact_threshold delay">
-        <ros2_control name="legged_unitree_hw" type="system">
+    <xacro:macro name="legged_ros2_control" params="hardware_plugin robot_type power_limit contact_threshold delay">
+        <ros2_control name="legged_hw" type="system">
             <hardware>
                 <plugin>${hardware_plugin}</plugin>

File: legged_robots/legged_description/urdf/p1/robot.xacro (robot description, xacro)
@@ -50,5 +50,5 @@
         <origin rpy="0 0 0" xyz="${-leg_offset_x} ${-leg_offset_y} 0"/>
     </xacro:leg_p1>
-    <xacro:legged_unitree_ros2_control hardware_plugin="$(arg hardware_plugin)"
+    <xacro:legged_ros2_control hardware_plugin="$(arg hardware_plugin)"
                                        robot_type="$(arg robot_type)"
                                        power_limit="$(arg power_limit)"

File: legged_robots/legged_description/urdf/robot.xacro (robot description, xacro)
@@ -50,5 +50,5 @@
         <origin rpy="0 0 0" xyz="${-leg_offset_x} ${-leg_offset_y} 0"/>
     </xacro:leg>
-    <xacro:legged_unitree_ros2_control hardware_plugin="$(arg hardware_plugin)"
+    <xacro:legged_ros2_control hardware_plugin="$(arg hardware_plugin)"
                                        robot_type="$(arg robot_type)"
                                        power_limit="$(arg power_limit)"

Commit message: [feat] P1 real hw interface

File: legged_robots/legged_description/urdf/common/ros2_control.xacro (robot description, xacro)
@@ -18,5 +18,5 @@
         </sensor>
     </xacro:macro>
-    <xacro:macro name="legged_ros2_control" params="hardware_plugin robot_type power_limit contact_threshold delay">
+    <xacro:macro name="legged_ros2_control" params="hardware_plugin robot_type power_limit contact_threshold delay command_mode:=10 dds_domain:=0 dds_state_topic:=p1_motor_state dds_imu_topic:=p1_imu dds_command_topic:=p1_motor_cmd dds_joint_order:=LF_HAA,LF_HFE,LF_KFE,LH_HAA,LH_HFE,LH_KFE,RF_HAA,RF_HFE,RF_KFE,RH_HAA,RH_HFE,RH_KFE contact_estimation_method:=current contact_force_threshold:=40.0 current_to_torque_scale:=1.0 current_to_torque_offset:=0.0">
         <ros2_control name="legged_hw" type="system">
             <hardware>
@@ -26,4 +26,14 @@
                 <param name="contact_threshold">${contact_threshold}</param>
                 <param name="delay">${delay}</param>
+                <param name="command_mode">${command_mode}</param>
+                <param name="dds_domain">${dds_domain}</param>
+                <param name="dds_state_topic">${dds_state_topic}</param>
+                <param name="dds_imu_topic">${dds_imu_topic}</param>
+                <param name="dds_command_topic">${dds_command_topic}</param>
+                <param name="dds_joint_order">${dds_joint_order}</param>
+                <param name="contact_estimation_method">${contact_estimation_method}</param>
+                <param name="contact_force_threshold">${contact_force_threshold}</param>
+                <param name="current_to_torque_scale">${current_to_torque_scale}</param>
+                <param name="current_to_torque_offset">${current_to_torque_offset}</param>
             </hardware>
             <xacro:legged_joint_ros2_control name="LF_HAA"/>

File: legged_robots/legged_description/urdf/p1/robot.xacro (robot description, xacro)
@@ -13,4 +13,14 @@
     <xacro:arg name="contact_threshold" default="40"/>
     <xacro:arg name="delay" default="0.009"/>
+    <xacro:arg name="command_mode" default="10"/>
+    <xacro:arg name="dds_domain" default="0"/>
+    <xacro:arg name="dds_state_topic" default="p1_motor_state"/>
+    <xacro:arg name="dds_imu_topic" default="p1_imu"/>
+    <xacro:arg name="dds_command_topic" default="p1_motor_cmd"/>
+    <xacro:arg name="dds_joint_order" default="LF_HAA,LF_HFE,LF_KFE,LH_HAA,LH_HFE,LH_KFE,RF_HAA,RF_HFE,RF_KFE,RH_HAA,RH_HFE,RH_KFE"/>
+    <xacro:arg name="contact_estimation_method" default="current"/>
+    <xacro:arg name="contact_force_threshold" default="40.0"/>
+    <xacro:arg name="current_to_torque_scale" default="1.0"/>
+    <xacro:arg name="current_to_torque_offset" default="0.0"/>
     <xacro:property name="mesh_path" value="file://$(find legged_description)/meshes/p1"/>
     <link name="base">
@@ -54,4 +64,14 @@
                                        power_limit="$(arg power_limit)"
                                        contact_threshold="$(arg contact_threshold)"
-                                       delay="$(arg delay)"/>
+                                       delay="$(arg delay)"
+                                       command_mode="$(arg command_mode)"
+                                       dds_domain="$(arg dds_domain)"
+                                       dds_state_topic="$(arg dds_state_topic)"
+                                       dds_imu_topic="$(arg dds_imu_topic)"
+                                       dds_command_topic="$(arg dds_command_topic)"
+                                       dds_joint_order="$(arg dds_joint_order)"
+                                       contact_estimation_method="$(arg contact_estimation_method)"
+                                       contact_force_threshold="$(arg contact_force_threshold)"
+                                       current_to_torque_scale="$(arg current_to_torque_scale)"
+                                       current_to_torque_offset="$(arg current_to_torque_offset)"/>
 </robot>

Commit message: [feat] Test dds remote control

File: legged_robots/legged_description/urdf/common/ros2_control.xacro (robot description, xacro)
@@ -18,5 +18,5 @@
         </sensor>
     </xacro:macro>
-    <xacro:macro name="legged_ros2_control" params="hardware_plugin robot_type power_limit contact_threshold delay command_mode:=10 dds_domain:=0 dds_state_topic:=p1_motor_state dds_imu_topic:=p1_imu dds_command_topic:=p1_motor_cmd dds_joint_order:=LF_HAA,LF_HFE,LF_KFE,LH_HAA,LH_HFE,LH_KFE,RF_HAA,RF_HFE,RF_KFE,RH_HAA,RH_HFE,RH_KFE contact_estimation_method:=current contact_force_threshold:=40.0 current_to_torque_scale:=1.0 current_to_torque_offset:=0.0">
+    <xacro:macro name="legged_ros2_control" params="hardware_plugin robot_type power_limit contact_threshold delay command_mode:=10 dds_domain:=0 dds_state_topic:=p1_motor_state dds_imu_topic:=p1_imu dds_command_topic:=p1_motor_cmd emergency_stop_topic:=/p1_emergency_stop dds_joint_order:=LF_HAA,LF_HFE,LF_KFE,LH_HAA,LH_HFE,LH_KFE,RF_HAA,RF_HFE,RF_KFE,RH_HAA,RH_HFE,RH_KFE contact_estimation_method:=current contact_force_threshold:=40.0 current_to_torque_scale:=1.0 current_to_torque_offset:=0.0">
         <ros2_control name="legged_hw" type="system">
             <hardware>
@@ -31,4 +31,5 @@
                 <param name="dds_imu_topic">${dds_imu_topic}</param>
                 <param name="dds_command_topic">${dds_command_topic}</param>
+                <param name="emergency_stop_topic">${emergency_stop_topic}</param>
                 <param name="dds_joint_order">${dds_joint_order}</param>
                 <param name="contact_estimation_method">${contact_estimation_method}</param>

File: legged_robots/legged_description/urdf/p1/robot.xacro (robot description, xacro)
@@ -18,8 +18,9 @@
     <xacro:arg name="dds_imu_topic" default="p1_imu"/>
     <xacro:arg name="dds_command_topic" default="p1_motor_cmd"/>
+    <xacro:arg name="emergency_stop_topic" default="/p1_emergency_stop"/>
     <xacro:arg name="dds_joint_order" default="LF_HAA,LF_HFE,LF_KFE,LH_HAA,LH_HFE,LH_KFE,RF_HAA,RF_HFE,RF_KFE,RH_HAA,RH_HFE,RH_KFE"/>
     <xacro:arg name="contact_estimation_method" default="current"/>
     <xacro:arg name="contact_force_threshold" default="40.0"/>
-    <xacro:arg name="current_to_torque_scale" default="1.0"/>
+    <xacro:arg name="current_to_torque_scale" default="2.863"/>
     <xacro:arg name="current_to_torque_offset" default="0.0"/>
     <xacro:property name="mesh_path" value="file://$(find legged_description)/meshes/p1"/>
@@ -70,4 +71,5 @@
                                        dds_imu_topic="$(arg dds_imu_topic)"
                                        dds_command_topic="$(arg dds_command_topic)"
+                                       emergency_stop_topic="$(arg emergency_stop_topic)"
                                        dds_joint_order="$(arg dds_joint_order)"
                                        contact_estimation_method="$(arg contact_estimation_method)"

Commit message: [feat] Tested with real lr_pro

File: legged_robots/legged_description/urdf/common/ros2_control.xacro (robot description, xacro)
@@ -18,5 +18,5 @@
         </sensor>
     </xacro:macro>
-    <xacro:macro name="legged_ros2_control" params="hardware_plugin robot_type power_limit contact_threshold delay command_mode:=10 dds_domain:=0 dds_state_topic:=p1_motor_state dds_imu_topic:=p1_imu dds_command_topic:=p1_motor_cmd emergency_stop_topic:=/p1_emergency_stop dds_joint_order:=LF_HAA,LF_HFE,LF_KFE,LH_HAA,LH_HFE,LH_KFE,RF_HAA,RF_HFE,RF_KFE,RH_HAA,RH_HFE,RH_KFE contact_estimation_method:=current contact_force_threshold:=40.0 current_to_torque_scale:=1.0 current_to_torque_offset:=0.0">
+    <xacro:macro name="legged_ros2_control" params="hardware_plugin robot_type power_limit contact_threshold delay delay_cycles:=9 command_mode:=10 dds_domain:=0 dds_state_topic:=p1_motor_state dds_imu_topic:=p1_imu dds_command_topic:=p1_motor_cmd emergency_stop_topic:=/p1_emergency_stop dds_joint_order:=LF_HAA,LF_HFE,LF_KFE,LH_HAA,LH_HFE,LH_KFE,RF_HAA,RF_HFE,RF_KFE,RH_HAA,RH_HFE,RH_KFE contact_estimation_method:=current contact_force_threshold:=40.0 current_to_torque_scale:=1.0 current_to_torque_offset:=0.0 feedforward_torque_slew_rate:=150.0 max_feedforward_torque:=0.0">
         <ros2_control name="legged_hw" type="system">
             <hardware>
@@ -26,4 +26,5 @@
                 <param name="contact_threshold">${contact_threshold}</param>
                 <param name="delay">${delay}</param>
+                <param name="delay_cycles">${delay_cycles}</param>
                 <param name="command_mode">${command_mode}</param>
                 <param name="dds_domain">${dds_domain}</param>
@@ -37,4 +38,6 @@
                 <param name="current_to_torque_scale">${current_to_torque_scale}</param>
                 <param name="current_to_torque_offset">${current_to_torque_offset}</param>
+                <param name="feedforward_torque_slew_rate">${feedforward_torque_slew_rate}</param>
+                <param name="max_feedforward_torque">${max_feedforward_torque}</param>
             </hardware>
             <xacro:legged_joint_ros2_control name="LF_HAA"/>

File: legged_robots/legged_description/urdf/p1/robot.xacro (robot description, xacro)
@@ -22,6 +22,8 @@
     <xacro:arg name="contact_estimation_method" default="current"/>
     <xacro:arg name="contact_force_threshold" default="40.0"/>
-    <xacro:arg name="current_to_torque_scale" default="2.863"/>
+    <xacro:arg name="current_to_torque_scale" default="1"/>
     <xacro:arg name="current_to_torque_offset" default="0.0"/>
+    <xacro:arg name="feedforward_torque_slew_rate" default="150.0"/>
+    <xacro:arg name="max_feedforward_torque" default="0.0"/>
     <xacro:property name="mesh_path" value="file://$(find legged_description)/meshes/p1"/>
     <link name="base">
@@ -76,4 +78,6 @@
                                        contact_force_threshold="$(arg contact_force_threshold)"
                                        current_to_torque_scale="$(arg current_to_torque_scale)"
-                                       current_to_torque_offset="$(arg current_to_torque_offset)"/>
+                                       current_to_torque_offset="$(arg current_to_torque_offset)"
+                                       feedforward_torque_slew_rate="$(arg feedforward_torque_slew_rate)"
+                                       max_feedforward_torque="$(arg max_feedforward_torque)"/>
 </robot>
